File: CAD/termoDaQ.sch (EAGLE design)
At the start: 59 parts, among them J1 SUPPLY, J10 POTENTIOMETER, J11 SUPPLY, J12 SUPPLY, J13 CONN_26X2, J14 CONN_26X2, J15 CONN_26X2, J16 CONN_26X2, J17 CONN_26X2, J18 CONN_26X2, J19 CONN_20X2, J2 ADC, J3 GPS, J4 SERIAL, J5 GPS ON/OF, J6 INT, J7 MPX, J8 SD, J9 EN, T1 2N2222, U1 328P, U2 DS18B20, U3 TINY85-20-DIP, Y1 16MHz, Y2 16MHz

Commit message: Source files update
Parts:
- added C18, C19: 22uF, SparkFun-Capacitors:10UF-POLAR-RADIAL-2.5MM-25V-20%
- added J20: VCC, SparkFun-Connectors:CONN_01
- added J21, J22, J23: CONN_26X2, SparkFun-Connectors:CONN_26X2
- added J24: CONN_20X2, SparkFun-Connectors:CONN_20X2
- added J25: FEMALE 2x3, SparkFun-Connectors:CONN_03X2FEMALE
- added S3: ON/OFF, SparkFun-Switches:SWITCH-SPDT-PTH-11.6X4.0MM
- J1: value SUPPLY -> TEST SUPPLY; device SparkFun-Connectors:CONN_023.5MM -> SparkFun-Connectors:CONN_02
- J13: value CONN_26X2 -> V+; device SparkFun-Connectors:CONN_26X2 -> SparkFun-Connectors:CONN_02
- J14: value CONN_26X2 -> B+; device SparkFun-Connectors:CONN_26X2 -> SparkFun-Connectors:CONN_02
- J15: value CONN_26X2 -> VCC; device SparkFun-Connectors:CONN_26X2 -> SparkFun-Connectors:CONN_02
- J16: value CONN_26X2 -> V-; device SparkFun-Connectors:CONN_26X2 -> SparkFun-Connectors:CONN_02
- J17: value CONN_26X2 -> B-; device SparkFun-Connectors:CONN_26X2 -> SparkFun-Connectors:CONN_02
- J18: value CONN_26X2 -> GND; device SparkFun-Connectors:CONN_26X2 -> SparkFun-Connectors:CONN_02
- J19: value CONN_20X2 -> SUPPLY; device SparkFun-Connectors:CONN_20X2 -> SparkFun-Connectors:CONN_025MM
Connections:
- new net N$13: J14.1, J14.2
- new net N$31: J17.1, J17.2
- new net N$32: J13.1, J13.2, J19.1
- new net N$33: J16.1, J16.2, J19.2
- new net V_BATT: J15.1, J15.2, J25.1, J25.2
- net 5V: now also C15.2, C18.+, C19.+, J10.5, J10.6, J11.1, J12.1, J24.10, J24.12, J24.14, J24.16, J24.18, J24.2, J24.20, J24.22, J24.24, J24.26, J24.28, J24.30, J24.32, J24.34, J24.36, J24.38, J24.4, J24.40, J24.6, J24.8, R10.1, R9.1, S3.P, U3.VCC
- net GND: now also C18.-, C19.-, J24.1, J24.11, J24.13, J24.15, J24.17, J24.19, J24.21, J24.23, J24.25, J24.27, J24.29, J24.3, J24.31, J24.33, J24.35, J24.37, J24.39, J24.5, J24.7, J24.9, J25.3, J25.4; no longer J13.1, J13.2, J14.1, J14.2, J15.1, J15.2, J16.1, J16.2, J17.1, J17.2, J19.1, J19.11, J19.13, J19.15, J19.17, J19.19, J19.21, J19.23, J19.25, J19.27, J19.29, J19.3, J19.31, J19.33, J19.35, J19.37, J19.39, J19.5, J19.7, J19.9
- net VCC: now also J20.1, J25.5, J25.6, S3.O; no longer C15.2, J10.5, J10.6, J11.1, J12.1, J13.3, J13.4, J14.3, J14.4, J15.3, J15.4, J16.3, J16.4, J17.3, J17.4, J18.3, J18.4, J19.10, J19.12, J19.14, J19.16, J19.18, J19.2, J19.20, J19.22, J19.24, J19.26, J19.28, J19.30, J19.32, J19.34, J19.36, J19.38, J19.4, J19.40, J19.6, J19.8, R10.1, R9.1, U3.VCC
Other:
- moved on the sheet: J1

Commit message: Source files, Update
Parts:
- added B+: B+, wirepad:SMD5
- added B-: B-, wirepad:SMD5
- added C20, C21, C22, C23, C28, C29, C31, C32, C33: 0.1uF, SparkFun-Capacitors:0.1UF-KIT-EZ-50V-20%
- added C24, C25: 22pF, SparkFun-Capacitors:22PF-PTH-2.54MM-200V-5%
- added C26, C27, C30: 10uF, SparkFun-Capacitors:10UF-POLAR-RADIAL-2.5MM-25V-20%
- added D5: PPS, SparkFun-LED:LED5MM
- added E-1, E-2, EN: EN GPS, wirepad:SMD2
- added G-1, G-2: G, wirepad:SMD2
- added GND: GND, wirepad:SMD2
- added INT: INT1, wirepad:SMD2
- added J26: OK, SparkFun-Connectors:CONN_03
- added J27: GND2, SparkFun-Connectors:CONN_01
- added J28: INT1, SparkFun-Connectors:CONN_01
- added J29: AIN, SparkFun-Connectors:CONN_03
- added J30: SERIAL, SparkFun-Connectors:CONN_06SILK_FEMALE_PTH
- added J31: GPS ON/OF, SparkFun-Connectors:CONN_03
- added J32, J35: GPS, SparkFun-Connectors:CONN_05
- added J33: TERMINAL SONDA, SparkFun-Connectors:CONN_03-SCREW-5MM
- added J34: GND, SparkFun-Connectors:CONN_01
- added J36: EN, SparkFun-Connectors:CONN_01
- added P-1, P-2: P, wirepad:SMD2
- added PPS: PPS, wirepad:SMD2
- added R-1, R-2: R, wirepad:SMD2
- added R12: 330, SparkFun-Resistors:330OHM-HORIZ-1/10W-5%
- added RX: RX, wirepad:SMD2
- added S4: STREAM, SparkFun-Switches:SWITCH-SPDT-PTH-11.6X4.0MM
- added T-1, T-2: T, wirepad:SMD2
- added TX: TX, wirepad:SMD2
- added V-1, V-2: V, wirepad:SMD2
- added VCC: VCC, wirepad:SMD2
- C1, C10, C13, C19: value 22uF -> 0.1uF; device SparkFun-Capacitors:10UF-POLAR-RADIAL-2.5MM-25V-20% -> SparkFun-Capacitors:0.1UF-KIT-EZ-50V-20%
- C12, C15, C4: value 0.1uF -> 10uF; device SparkFun-Capacitors:0.1UF-KIT-EZ-50V-20% -> SparkFun-Capacitors:10UF-POLAR-RADIAL-2.5MM-25V-20%
- C16, C8: value 22pF -> 0.1uF; device SparkFun-Capacitors:22PF-PTH-2.54MM-200V-5% -> SparkFun-Capacitors:0.1UF-KIT-EZ-50V-20%
- C17: value 22pF -> 10uF; device SparkFun-Capacitors:22PF-PTH-2.54MM-200V-5% -> SparkFun-Capacitors:10UF-POLAR-RADIAL-2.5MM-25V-20%
- C18, C2, C3: value 22uF -> 10uF
- C6: value 0.1uF -> 22pF; device SparkFun-Capacitors:0.1UF-KIT-EZ-50V-20% -> SparkFun-Capacitors:22PF-PTH-2.54MM-200V-5%
- D1: value PROG -> ON
- D2: value PPS -> POWER; device SparkFun-LED:LED5MM -> SparkFun-LED:LED3MM
- D3: value ERROR -> PROG
- D4: value ON -> ERROR
- J1: value TEST SUPPLY -> JUMPER EN; device SparkFun-Connectors:CONN_02 -> SparkFun-Connectors:CONN_03
- J10: value POTENTIOMETER -> LED ON/OFF; device SparkFun-Connectors:CONN_03X2FEMALE -> SparkFun-Connectors:CONN_03
- J12: value SUPPLY -> STEP UP; device SparkFun-Connectors:CONN_023.5MM -> SparkFun-Connectors:CONN_03
- J13: value V+ -> B+
- J14: value B+ -> GND
- J16: value V- -> B-
- J17: value B- -> MPX EXT; device SparkFun-Connectors:CONN_02 -> SparkFun-Connectors:CONN_03
- J18: value GND -> MPX; device SparkFun-Connectors:CONN_02 -> SparkFun-Connectors:CONN_06SILK_FEMALE_PTH
- J19: value SUPPLY -> E_AD2; device SparkFun-Connectors:CONN_025MM -> SparkFun-Connectors:CONN_01
- J2: value ADC -> G; device SparkFun-Connectors:CONN_05 -> SparkFun-Connectors:CONN_01
- J20: value VCC -> SD; device SparkFun-Connectors:CONN_01 -> SparkFun-Connectors:CONN_07
- J21: value CONN_26X2 -> ADC; device SparkFun-Connectors:CONN_26X2 -> SparkFun-Connectors:CONN_05
- J22: value CONN_26X2 -> I2C; device SparkFun-Connectors:CONN_26X2 -> SparkFun-Connectors:CONN_04
- J23: value CONN_26X2 -> MODULO SD; device SparkFun-Connectors:CONN_26X2 -> SparkFun-Connectors:CONN_06POLAR
- J24: value CONN_20X2 -> V+; device SparkFun-Connectors:CONN_20X2 -> SparkFun-Connectors:CONN_02
- J25: value FEMALE 2x3 -> V-; device SparkFun-Connectors:CONN_03X2FEMALE -> SparkFun-Connectors:CONN_02
- J3: value GPS -> FEMALE 2x3; device SparkFun-Connectors:CONN_06SILK_FEMALE_PTH -> SparkFun-Connectors:CONN_03X2FEMALE
- J4: value SERIAL -> BETERIA; device SparkFun-Connectors:CONN_06SILK_FEMALE_PTH -> SparkFun-Connectors:CONN_02
- J5: value GPS ON/OF -> INT2; device SparkFun-Connectors:CONN_03 -> SparkFun-Connectors:CONN_01
- J6: value INT -> EN
- J7: value MPX -> TEST SUPPLY; device SparkFun-Connectors:CONN_06SILK_FEMALE_PTH -> SparkFun-Connectors:CONN_02
- J8: value SD -> GND; device SparkFun-Connectors:CONN_07 -> SparkFun-Connectors:CONN_01
- J9: value EN -> GND; device SparkFun-Connectors:CONN_01 -> SparkFun-Connectors:CONN_02
- R1: value 10k -> 330; device SparkFun-Resistors:10KOHM-HORIZ-1/4W-5% -> SparkFun-Resistors:330OHM-HORIZ-1/10W-5%
- R10: value 4.7k -> 1k; SPICEPREFIX (none) -> R
- R2, R3, R9: value 330 -> 1k; device SparkFun-Resistors:330OHM-HORIZ-1/10W-5% -> SparkFun-Resistors:1KOHM-HORIZ-1/4W-1%
- R6: value 1k -> 330; device SparkFun-Resistors:1KOHM-HORIZ-1/4W-1% -> SparkFun-Resistors:330OHM-HORIZ-1/10W-5%
- R7: value 1k -> 10k; device SparkFun-Resistors:1KOHM-HORIZ-1/4W-1% -> SparkFun-Resistors:10KOHM-HORIZ-1/4W-5%
- R8: value 4.7k -> 330; device SparkFun-Resistors:1KOHM-HORIZ-1/4W-1% -> SparkFun-Resistors:330OHM-HORIZ-1/10W-5%
- S1: value RESET -> ON/OFF; device SparkFun-Switches:MOMENTARY-SWITCH-SPST-PTH-6.0MM -> SparkFun-Switches:SWITCH-SPDT-PTH-11.6X4.0MM
- S2: value STREAM -> ON/OFF
- S3: value ON/OFF -> RESET; device SparkFun-Switches:SWITCH-SPDT-PTH-11.6X4.0MM -> SparkFun-Switches:MOMENTARY-SWITCH-SPST-PTH-6.0MM
- U1: value 328P -> TINY85-20-DIP; device SparkFun-IC-Microcontroller:ATMEGA328P_PDIP -> SparkFun-Retired:ATTINY45TINY85-20-DIP
- U2: value DS18B20 -> 328P; device SparkFun-Sensors:DS18B20 -> SparkFun-IC-Microcontroller:ATMEGA328P_PDIP
- U3: value TINY85-20-DIP -> DS18B20; device SparkFun-Retired:ATTINY45TINY85-20-DIP -> SparkFun-Sensors:DS18B20
Connections:
- removed net AD1: J2.1, U1.PC1(ADC1)
- removed net N$1: C8.1, U1.PB7(XTAL2/TOSC2), Y1.2
- removed net N$10: D3.A, U1.PD3(INT1)
- removed net N$11: J10.3, J10.4, U3.PB0(MOSI)
- removed net N$13: J14.1, J14.2
- removed net N$14: C17.1, U3.PB3(ADC3), Y2.2
- removed net N$15: R8.1, U1.PD5(T1), U2.DQ
- removed net N$18: J4.2, U1.PD0(RXD)
- removed net N$19: J4.3, U1.PD1(TXD)
- removed net N$2: C5.1, U1.PB6(XTAL1/TOSC1), Y1.1
- removed net N$21: J6.1, R4.1, U1.PD2(INT0)
- removed net N$22: R11.2, U3.PB2(SCK/ADC1)
- removed net N$23: C16.1, U3.PB4(ADC2), Y2.1
- removed net N$24: D4.A, R9.2
- removed net N$25: J5.2, U1.PD6(AIN0)
- removed net N$3: C7.2, U1.AREF
- removed net N$31: J17.1, J17.2
- removed net N$32: J13.1, J13.2, J19.1
- removed net N$33: J16.1, J16.2, J19.2
- removed net N$4: C9.1, R1.1, S1.1, U1.PC6(/RESET)
- removed net N$5 (its old number): D1.C, R2.1
- removed net N$6: R10.2, U3.PB5(NRES)
- removed net N$7: J9.1, U3.PB1(MISO)
- removed net N$9: C11.1, J7.1, U1.PC0(ADC0)
- new net /RESET: C32.1, R7.1, S3.1, U2.PC6(/RESET)
- new net AREF: C21.2, U2.AREF
- new net B+: C13.1, C16.1, J13.1, J13.2, S2.P
- new net B+IN: B+.P, J4.1, S2.S
- new net B-: B-.P, C13.2, C16.2, J16.1, J16.2, J4.2
- new net DS18B20: J33.2, R9.1, U2.PD5(T1), U3.DQ
- new net ERROR: D4.A, U2.PD3(INT1)
- new net GND2: J23.1, J27.1, J29.1, J33.3
- new net INT1: INT.P, J28.1, R6.1, U2.PD2(INT0)
- new net INT2: J26.2, J26.3, J5.1, U1.PB1(MISO)
- new net JA_LED: J10.2, J10.3, R4.1
- new net J_EN: J1.1, J6.1, R3.2, U1.PB0(MOSI)
- new net MPX: C20.1, J17.1, J18.1, U2.PC0(ADC0)
- new net M_XTAL1: C24.1, U2.PB6(XTAL1/TOSC1), Y2.1
- new net M_XTAL2: C25.1, U2.PB7(XTAL2/TOSC2), Y2.2
- new net N$12: D4.C, R8.1
- new net NRES: R2.2, U1.PB5(NRES)
- new net OK: J26.1, U2.PD7(AIN1)
- new net POT: J3.3, J3.4, U1.PB2(SCK/ADC1)
- new net PWR_LED1: D2.A, R4.2
- new net PWR_LED2: D1.A, R1.2
- new net R/GPS: J31.2, U2.PD6(AIN0)
- new net RX: J30.3, U2.PD0(RXD)
- new net TX: J30.2, U2.PD1(TXD)
- new net V+: J24.1, J24.2
- new net V-: J25.1, J25.2
- new net XTAL1: C6.2, U1.PB4(ADC2), Y1.2
- new net XTAL2: C5.1, U1.PB3(ADC3), Y1.1
- net 5V: now also C1.2, C12.+, C15.+, C17.+, C19.2, C22.1, C23.2, C26.+, C27.+, C28.1, C30.+, C31.1, C33.1, C9.2, J10.1, J17.3, J18.3, J20.4, J22.2, J23.2, J29.2, J3.5, J3.6, J30.4, J31.3, J32.2, J33.1, J35.2, J7.1, R1.1, R2.1, R6.2, R7.2, R9.2, S1.P, S4.O, U2.AVCC, U2.VCC, U3.VDD, V-1.P, V-2.P, VCC.P; no longer C1.+, C10.+, C12.2, C13.+, C15.2, C19.+, C2.+, C4.1, C6.2, J1.1, J10.5, J10.6, J12.1, J24.10, J24.12, J24.14, J24.16, J24.18, J24.2, J24.20, J24.22, J24.24, J24.26, J24.28, J24.30, J24.32, J24.34, J24.36, J24.38, J24.4, J24.40, J24.6, J24.8, J3.2, J4.4, J5.3, J7.3, J8.4, R1.2, R10.1, R4.2, R8.2, R9.1, S2.O, S3.P, U1.AVCC, U2.VDD, U3.VCC
- net AD2: now also J19.1, J21.2, U2.PC2(ADC2); no longer J2.2, U1.PC2(ADC2)
- net AD3: now also J21.3, J29.3, U2.PC3(ADC3); no longer J2.3, U1.PC3(ADC3)
- net AD4: now also J21.4, J22.3, U2.PC4(ADC4/SDA); no longer J2.4, U1.PC4(ADC4/SDA)
- net AD5: now also J21.5, J22.4, U2.PC5(ADC5/SCL); no longer J2.5, U1.PC5(ADC5/SCL)
- net CD: now also J20.1, J23.6, U2.PB2(SS/OC1B); no longer J8.1, U1.PB2(SS/OC1B)
- net CLK: now also D3.A, J20.5, J23.5, U2.PB5(SCK); no longer D1.A, J8.5, U1.PB5(SCK)
- net CMD: now also J20.2, J23.4, U2.PB3(MOSI/OC2); no longer J8.2, U1.PB3(MOSI/OC2)
- net DAT: now also J20.7, J23.3, U2.PB4(MISO); no longer J8.7, U1.PB4(MISO)
- net DTR: now also C32.2, J30.1; no longer C9.2, J4.1
- net EN: now also C29.1, E-1.P, E-2.P, EN.P, J1.2, J1.3, J36.1; no longer J3.6, U1.PD7(AIN1)
- net GND: now also C1.1, C10.2, C12.-, C15.-, C17.-, C19.1, C20.2, C21.1, C22.2, C23.1, C24.2, C25.2, C26.-, C27.-, C28.2, C29.2, C30.-, C31.2, C33.2, C4.-, C7.2, C9.1, D1.C, D2.C, G-1.P, G-2.P, GND.P, J14.1, J14.2, J17.2, J2.1, J20.3, J20.6, J22.1, J3.1, J3.2, J30.5, J30.6, J32.5, J34.1, J35.5, J8.1, J9.1, J9.2, R10.2, R11.2, R12.1, R8.2, S3.2, U1.GND, U2.GND@1, U2.GND@2; no longer C1.-, C10.-, C12.1, C13.-, C15.1, C16.2, C17.2, C19.-, C4.2, C7.1, D4.C, J1.2, J10.1, J10.2, J18.1, J24.1, J24.11, J24.13, J24.15, J24.17, J24.19, J24.21, J24.23, J24.25, J24.27, J24.29, J24.3, J24.31, J24.33, J24.35, J24.37, J24.39, J24.5, J24.7, J24.9, J25.3, J25.4, J3.5, J4.5, J4.6, J8.3, J8.6, R2.2, R3.1, R6.2, R7.2, S1.2, U1.GND@1, U1.GND@2, U2.GND
- net N$16: now also J31.1, R11.1; no longer J5.1, R7.1
- net N$17: now also R10.1, S4.S; no longer R6.1, S2.S
- net N$20: now also R3.1; no longer R11.1
- net N$8: now also D5.C, R12.2; no longer D2.C, R3.2
- net PC: now also S4.P, U2.PD4(XCK/T0); no longer S2.P, U1.PD4(XCK/T0)
- net PPS: now also D5.A, J32.1, J35.1, P-1.P, P-2.P, PPS.P; no longer D2.A, J3.1
- net R: now also J32.4, J35.4, R-1.P, R-2.P, RX.P, U2.PB1(OC1A); no longer J3.4, U1.PB1(OC1A)
- net T: now also J32.3, J35.3, T-1.P, T-2.P, TX.P, U2.PB0(ICP); no longer J3.3, U1.PB0(ICP)
- net VCC: now also C11.1, C2.+, C8.1, J12.3, S1.O; no longer J20.1, J25.5, J25.6, S3.O
- net V_BATT: now also C10.1, C4.+, C7.1, J12.1, J21.1, U2.PC1(ADC1); no longer J25.1, J25.2
Other:
- note added: "ATMEGA328P"
- note added: "ATTINY85"
- note added: "BATERIA"
- note added: "Creative Commons Attribution-ShareAlike 4.0"
- note added: "DS18B20"
- note added: "ERROR LED"
- note added: "FILTRO"
- note added: "FUENTE"
- note added: "GPS"
- note added: "HEADERS"
- note added: "JESUS ALFONSO RODRIGUEZ LISTA"
- note added: "MPX5700"
- note added: "PROG LED"
- note added: "SD"
- note added: "[OSHW]VE000001"
- note added: "github.com/mc-ireiser/termoDaQ"
- note added: "termoDaQ V1.0"
